File: KiCAD/bp-chipcon/keypad.sch (KiCad schematic (older format))
At the start: 20 parts, among them J3 KEYPAD connector, SW2 A, SW3 C, SW4 B, SW5 D, SW6 RIGHT, SW7 DOWN, SW8 LEFT, SW9 UP, U2 74HC164N

Commit message: Modification to schematic
Parts:
- renumbered D11 to D10, D12 to D11, D5 to D4, D6 to D5, D7 to D6, D8 to D7, D9 to D8, D10 to D9, J3 to J4
Changed lines of the file:
@@
 $EndComp
 $Comp
-L device:D D7
+L device:D D6
 U 1 1 5CE42379
 P 5475 4525
-F 0 "D7" H 5475 4741 50  0000 C CNN
+F 0 "D6" H 5475 4741 50  0000 C CNN
 F 1 "1N4148" H 5475 4650 50  0000 C CNN
 F 2 "" H 5475 4525 50  0001 C CNN
@@
 $EndComp
 $Comp
-L device:D D8
+L device:D D7
 U 1 1 5CE42417
 P 5475 4875
-F 0 "D8" H 5475 5091 50  0000 C CNN
+F 0 "D7" H 5475 5091 50  0000 C CNN
 F 1 "1N4148" H 5475 5000 50  0000 C CNN
 F 2 "" H 5475 4875 50  0001 C CNN
@@
 $EndComp
 $Comp
-L device:D D9
+L device:D D8
 U 1 1 5CE4257A
 P 5475 5200
-F 0 "D9" H 5475 5416 50  0000 C CNN
+F 0 "D8" H 5475 5416 50  0000 C CNN
 F 1 "1N4148" H 5475 5325 50  0000 C CNN
 F 2 "" H 5475 5200 50  0001 C CNN
@@
 $EndComp
 $Comp
-L device:D D10
+L device:D D9
 U 1 1 5CE42581
 P 5475 5550
-F 0 "D10" H 5475 5766 50  0000 C CNN
+F 0 "D9" H 5475 5766 50  0000 C CNN
 F 1 "1N4148" H 5475 5675 50  0000 C CNN
 F 2 "" H 5475 5550 50  0001 C CNN
@@
 $EndComp
 $Comp
-L device:D D5
+L device:D D4
 U 1 1 5CE4260D
 P 5475 3825
-F 0 "D5" H 5475 4041 50  0000 C CNN
+F 0 "D4" H 5475 4041 50  0000 C CNN
 F 1 "1N4148" H 5475 3950 50  0000 C CNN
 F 2 "" H 5475 3825 50  0001 C CNN
@@
 $EndComp
 $Comp
-L device:D D6
+L device:D D5
 U 1 1 5CE42614
 P 5475 4175
-F 0 "D6" H 5475 4391 50  0000 C CNN
+F 0 "D5" H 5475 4391 50  0000 C CNN
 F 1 "1N4148" H 5475 4300 50  0000 C CNN
 F 2 "" H 5475 4175 50  0001 C CNN
@@
 	4650 5050 4650 5550
 $Comp
-L device:D D11
+L device:D D10
 U 1 1 5CE42A3D
 P 5475 5900
-F 0 "D11" H 5475 6116 50  0000 C CNN
+F 0 "D10" H 5475 6116 50  0000 C CNN
 F 1 "1N4148" H 5475 6025 50  0000 C CNN
 F 2 "" H 5475 5900 50  0001 C CNN
@@
 $EndComp
 $Comp
-L device:D D12
+L device:D D11
 U 1 1 5CE42A44
 P 5475 6250
-F 0 "D12" H 5475 6466 50  0000 C CNN
+F 0 "D11" H 5475 6466 50  0000 C CNN
 F 1 "1N4148" H 5475 6375 50  0000 C CNN
 F 2 "" H 5475 6250 50  0001 C CNN
@@
 	5625 4875 5625 4525
 $Comp
-L conn:Conn_01x05_Male J3
+L conn:Conn_01x05_Male J4
 U 1 1 5CE44CE8
 P 5000 2675
-F 0 "J3" V 5060 2915 50  0000 L CNN
+F 0 "J4" V 5060 2915 50  0000 L CNN
 F 1 "KEYPAD connector" V 4925 2350 50  0000 L CNN
 F 2 "" H 5000 2675 50  0001 C CNN
@@
 $EndComp
 $Comp
-L power:GND #PWR013
+L power:GND #PWR016
 U 1 1 5CE46111
 P 5200 2875
-F 0 "#PWR013" H 5200 2625 50  0001 C CNN
+F 0 "#PWR016" H 5200 2625 50  0001 C CNN
 F 1 "GND" H 5205 2702 50  0000 C CNN
 F 2 "" H 5200 2875 50  0001 C CNN
@@
 $EndComp
 Text Label 4775 3000 2    50   ~ 0
-+3.3v
++3.0v
 Wire Wire Line
 	4800 2875 4800 3000
@@
 IN
 Text Label 3400 4200 2    50   ~ 0
-+3.3v
++3.0v
 Text Label 3400 4550 2    50   ~ 0
-+3.3v
++3.0v
 Text HLabel 5200 2875 2    50   UnSpc ~ 0
 KEY_GND
@@
 $EndComp
 $Comp
-L power:GND #PWR0102
+L power:GND #PWR017
 U 1 1 5CE4CA9A
 P 2400 3000
-F 0 "#PWR0102" H 2400 2750 50  0001 C CNN
+F 0 "#PWR017" H 2400 2750 50  0001 C CNN
 F 1 "GND" H 2405 2827 50  0000 C CNN
 F 2 "" H 2400 3000 50  0001 C CNN
@@
 Connection ~ 5825 3825
 Text Label 5825 3525 2    50   ~ 0
-+3.3v
++3.0v
 $EndSCHEMATC

Commit message: work on tvout
Connections:
- net KEY_IN renamed KEY_DIN
- net KEY_OUT renamed KEY_DOUT
Changed lines of the file:
@@
 KEY_CLK
 Text HLabel 4750 3225 2    50   Output ~ 0
-KEY_OUT
+KEY_DOUT
 Text HLabel 4775 3125 2    50   Input ~ 0
-KEY_IN
+KEY_DIN
 $Comp
 L switches:SW_Push SW2
