File: KiCAD/bp-chipcon/bp-chipcon.sch (KiCad schematic (older format))
At the start: 33 parts, among them J1 audio_out, J2 video_out, J3 KEYPAD connector, M1 BLUE_PILL, Q1 2N3904, Q2 2N3906, SW1 power, U1 74HC86N

Commit message: Rework of tvout.c added video demo on youtube
Parts:
- R5: value 680 -> 620
Changed lines of the file:
@@
 P 8975 2050
 F 0 "R5" V 8768 2050 50  0000 C CNN
-F 1 "680" V 8859 2050 50  0000 C CNN
+F 1 "620" V 8859 2050 50  0000 C CNN
 F 2 "" V 8905 2050 50  0001 C CNN
 F 3 "" H 8975 2050 50  0001 C CNN
